File: kicad/PowerSupply-MotorDriver/PowerSupply-MotorDriver.sch (KiCad schematic (older format))
At the start: 9 parts

Commit message: Добавил дополнительные компоненты в схеме стабилизатора напряжения.
Parts:
- added FU1, FU2: 10 А, ~, symbol PROTECTOR
- added R1: 10 к, ~, symbol RESISTOR_1W
Connections:
- net at VD3.1, VD4.2: now also FU2.2; no longer XS1.2
- net at C1.1, C2.1, C3.1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: now also R1.2
- net at VD1.1, VD2.2: now also FU1.2; no longer XS1.1
- net at C1.2, C2.2, C3.2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: now also R1.1
- new net: FU1.1, XS1.1
- new net: FU2.1, XS1.2
Other:
- moved on the sheet: XS1, XS2
Changed lines of the file:
@@
 Sheet 1 1
 Title ""
-Date "4 dec 2015"
+Date "9 dec 2015"
 Rev ""
 Comp ""
@@
 	4600 3650 4600 3750
 Wire Wire Line
-	4200 3750 4800 3750
+	4300 3750 4600 3750
+Wire Wire Line
+	4600 3750 4700 3750
+Wire Wire Line
+	4700 3750 4800 3750
 Wire Wire Line
 	4800 3750 4800 3650
@@
 	5350 3650 5350 3750
 Wire Wire Line
-	5350 3750 5550 3750
+	5350 3750 5450 3750
+Wire Wire Line
+	5450 3750 5550 3750
 Wire Wire Line
 	5550 3750 5550 3650
 Connection ~ 4700 3750
 Wire Wire Line
-	5450 3750 5450 3950
+	5450 3750 5450 3850
+Wire Wire Line
+	5450 3850 5450 3950
 Connection ~ 5450 3750
 Wire Wire Line
 	4600 4350 4600 4450
 Wire Wire Line
-	4600 4450 5550 4450
+	4600 4450 4800 4450
+Wire Wire Line
+	4800 4450 5050 4450
+Wire Wire Line
+	5050 4450 5350 4450
+Wire Wire Line
+	5350 4450 5550 4450
 Wire Wire Line
 	5550 4450 5550 4350
@@
 	4700 3250 4700 3150
 Wire Wire Line
-	4700 3150 5450 3150
+	4700 3150 5050 3150
+Wire Wire Line
+	5050 3150 5450 3150
 Wire Wire Line
 	5450 3150 5450 3250
@@
 L PIN_F_2 XS1
 U 1 1 566197BD
-P 4200 3750
-F 0 "XS1" H 4350 3950 50  0000 L BNN
-F 1 "DG126-5.0-02P-14" H 4000 3850 50  0000 L BNN
-F 2 "~" H 4650 3900 50  0001 C CNN
-F 3 "" H 4200 3750 60  0000 C CNN
-	1    4200 3750
+P 3600 3850
+F 0 "XS1" H 3750 4050 50  0000 L BNN
+F 1 "DG126-5.0-02P-14" H 3400 3950 50  0000 L BNN
+F 2 "~" H 4050 4000 50  0001 C CNN
+F 3 "" H 3600 3850 60  0000 C CNN
+	1    3600 3850
 	-1   0    0    -1
 $EndComp
 Wire Wire Line
-	4200 3850 4400 3850
-Wire Wire Line
-	4400 3850 4400 4550
+	4400 4050 4400 4550
 Wire Wire Line
 	4950 3850 4950 4550
@@
 	5050 4450 5050 4550
 Wire Wire Line
-	5050 4550 7100 4550
+	5050 4550 6000 4550
+Wire Wire Line
+	6000 4550 6450 4550
+Wire Wire Line
+	6450 4550 6900 4550
+Wire Wire Line
+	6900 4550 7300 4550
+Wire Wire Line
+	7300 4550 7550 4550
 Connection ~ 5050 4450
 Wire Wire Line
-	5050 3050 7100 3050
+	5050 3050 6000 3050
+Wire Wire Line
+	6000 3050 6450 3050
+Wire Wire Line
+	6450 3050 6900 3050
+Wire Wire Line
+	6900 3050 7300 3050
+Wire Wire Line
+	7300 3050 7550 3050
 $Comp
 L CAPITORS_ELECTROLYTIC C1
@@
 L PIN_F_2 XS2
 U 1 1 56619A9C
-P 7200 3700
-F 0 "XS2" H 7450 3900 50  0000 L BNN
-F 1 "DG126-5.0-02P-14" H 7150 3800 50  0000 L BNN
-F 2 "~" H 7650 3850 50  0001 C CNN
-F 3 "" H 7200 3700 60  0000 C CNN
-	1    7200 3700
+P 7650 3700
+F 0 "XS2" H 7900 3900 50  0000 L BNN
+F 1 "DG126-5.0-02P-14" H 7600 3800 50  0000 L BNN
+F 2 "~" H 8100 3850 50  0001 C CNN
+F 3 "" H 7650 3700 60  0000 C CNN
+	1    7650 3700
 	1    0    0    -1
 $EndComp
 Wire Wire Line
-	7200 3700 7100 3700
-Wire Wire Line
-	7100 3700 7100 3050
+	7650 3700 7550 3700
+Wire Wire Line
+	7550 3700 7550 3050
 Connection ~ 6900 3050
 Wire Wire Line
-	7200 3800 7100 3800
-Wire Wire Line
-	7100 3800 7100 4550
+	7650 3800 7550 3800
+Wire Wire Line
+	7550 3800 7550 4550
 Connection ~ 6900 4550
+$Comp
+L PROTECTOR FU1
+U 1 1 5666E4C7
+P 4050 3750
+F 0 "FU1" H 4050 3850 60  0000 C CNN
+F 1 "10 А" H 4300 3850 60  0000 C CNN
+F 2 "~" H 4050 3750 60  0000 C CNN
+F 3 "~" H 4050 3750 60  0000 C CNN
+	1    4050 3750
+	1    0    0    -1
+$EndComp
+$Comp
+L PROTECTOR FU2
+U 1 1 5666E4F2
+P 4050 4050
+F 0 "FU2" H 4050 3950 60  0000 C CNN
+F 1 "10 А" H 4300 3950 60  0000 C CNN
+F 2 "~" H 4050 4050 60  0000 C CNN
+F 3 "~" H 4050 4050 60  0000 C CNN
+	1    4050 4050
+	1    0    0    1
+$EndComp
+Wire Wire Line
+	4400 4050 4300 4050
+Wire Wire Line
+	3600 3850 3850 3850
+Wire Wire Line
+	3850 3850 3850 3750
+Wire Wire Line
+	3850 3750 4050 3750
+Wire Wire Line
+	4050 4050 3850 4050
+Wire Wire Line
+	3850 4050 3850 3950
+Wire Wire Line
+	3850 3950 3600 3950
+$Comp
+L RESISTOR_1W R1
+U 1 1 566842DA
+P 7300 3900
+F 0 "R1" H 7400 4100 71  0000 C CNN
+F 1 "10 к" H 7400 4000 71  0000 C CNN
+F 2 "~" H 7300 3900 60  0000 C CNN
+F 3 "~" H 7300 3900 60  0000 C CNN
+	1    7300 3900
+	0    -1   -1   0
+$EndComp
+Wire Wire Line
+	7300 3050 7300 3650
+Connection ~ 7300 3050
+Wire Wire Line
+	7300 3900 7300 4550
+Connection ~ 7300 4550
 $EndSCHEMATC
